Commit message: Fix merge

File: test/integration/fixed_joint_reduction_visual.urdf (robot description, URDF)
Before this commit: robot fixed_joint_reduction_test_odel, 3 links, 2 joints
Links:
- added link link1a, mass 100
- added link link2, mass 200; visual box size=0.3 0.3 2.0
- added link link2a, mass 200; visual box size=0.3 0.3 2.0
- added link link3, mass 400; visual box size=0.3 0.4 0.5
- added link link3a, mass 400; visual box size=0.3 0.4 0.5
Joints:
- added joint joint01a: type continuous, parent link0, child link1a, origin xyz=0 0 -1 rpy=0 0 1.57079632679, axis 1 0 0
- added joint joint12: type revolute, parent link1, child link2, origin xyz=0 -3.0 0.0 rpy=-1.57079632679 0 -1.57079632679, axis 0 1 0, limit lower=0 upper=0 effort=10000 velocity=1000
- added joint joint12a: type fixed, parent link1a, child link2a, origin xyz=0 -3.0 0.0 rpy=-1.57079632679 0 -1.57079632679, axis 0 1 0, limit lower=0 upper=0 effort=10000 velocity=1000
- added joint joint23: type revolute, parent link2, child link3, origin xyz=-0.5 0.5 2.5 rpy=-1.57079632679 0 -1.57079632679, axis 0 1 0, limit lower=0 upper=0 effort=10000 velocity=1000
- added joint joint23a: type fixed, parent link2a, child link3a, origin xyz=-0.5 0.5 2.5 rpy=-1.57079632679 0 -1.57079632679, axis 0 1 0, limit lower=0 upper=0 effort=10000 velocity=1000
