Commit message: Test URDF continuous joint effort/velocity limits
Test currently fails.

Signed-off-by: Steve Peters <scpeters@openrobotics.org>

File: test/integration/urdf_joint_parameters.urdf (robot description, URDF)
Before this commit: robot urdf_joint_parameters, 6 links, 5 joints
Joints:
- joint joint01: limit (none) -> effort=1.0 velocity=1.0
- joint jointw0: limit (none) -> effort=0.0 velocity=0.0
