Commit message: Improve code coverage
Signed-off-by: Steve Peters <scpeters@openrobotics.org>

File: test/integration/fixed_joint_reduction_joint_frame_extension.urdf (robot description, URDF)
Before this commit: robot chained_fixed_joint_links, 4 links, 3 joints
Links:
- added link link4, mass 1; collision box size=1.0 1.0 1; visual box size=0.1 0.1 1
Joints:
- added joint joint4: type fixed, parent link3, child link4, origin xyz=0 1.0 0.0 rpy=0 0 0.7854
