Commit message: urdf_gazebo_extensions.urdf: remove joint23 since it creates a kinematic loop

File: test/integration/urdf_gazebo_extensions.urdf (robot description, URDF)
Before this commit: robot urdf_gazebo_extension_test, 6 links, 6 joints
Joints:
- removed joint joint23

Commit message: Backport test for URDF sensor poses
Backported from #525.

Signed-off-by: Steve Peters <scpeters@openrobotics.org>

File: test/integration/urdf_gazebo_extensions.urdf (robot description, URDF)
Before this commit: robot urdf_gazebo_extension_test, 6 links, 6 joints
Links:
- added link Camera, mass 0.10621
- added link issue378_link
- added link linkSensorNoPose, mass 100
- added link linkSensorPose, mass 100
- added link linkSensorPoseRelative, mass 100
- added link linkSensorPoseTwoLevel, mass 100
- added link linkSensorPoseTwoLevel2, mass 100
Joints:
- added joint issue378_link_joint: type fixed, parent link0, child issue378_link, origin xyz=0 0 0 rpy=0 -0 0, axis 0 0 0
- added joint jCamera: type fixed, parent link0, child Camera, origin xyz=-0.20115 0.42488 0.30943 rpy=1.5708 -0.89012 1.5708, axis 0 0 0
- added joint jointSensorNoPose: type fixed, parent link0, child linkSensorNoPose, origin xyz=333 0 0 rpy=0 0 1.57079632679
- added joint jointSensorPose: type fixed, parent link0, child linkSensorPose, origin xyz=333 0 0 rpy=0 0 1.57079632679
- added joint jointSensorPoseRelative: type fixed, parent link0, child linkSensorPoseRelative, origin xyz=333 0 0 rpy=0 0 1.57079632679
- added joint jointSensorPoseTwoLevel: type fixed, parent link0, child linkSensorPoseTwoLevel, origin xyz=0 0 222 rpy=0 0 0
- added joint jointSensorPoseTwoLevel2: type fixed, parent linkSensorPoseTwoLevel, child linkSensorPoseTwoLevel2, origin xyz=333 0 0 rpy=0 0 1.57079632679

Commit message: urdf extension test: fix URDF kinematics
The urdf_gazebo_extensions.urdf file had incorrect kinematics
with link3 being the child of two different joints.
This adds a link4 and converts joint13 to joint14.
This also fixes some expectations about the
implicit_spring_damper tags.

Signed-off-by: Steve Peters <scpeters@openrobotics.org>

File: test/integration/urdf_gazebo_extensions.urdf (robot description, URDF)
Before this commit: robot urdf_gazebo_extension_test, 13 links, 13 joints
Links:
- added link link4, mass 400; visual box size=0.3 0.4 0.5
Joints:
- removed joint joint13
- added joint joint14: type revolute, parent link1, child link4, origin xyz=0 -3.0 0.0 rpy=-1.57079632679 0 -1.57079632679, axis 0 1 0, limit lower=0 upper=0 effort=10000 velocity=1000
